Commit message: Update URDF files

File: urdf/car_control.urdf (robot description, URDF)
Before this commit: robot toy_car_3, 5 links, 4 joints
Links:
- removed link BR_coord
- added link BR_wheel, mass 2.8186; collision mesh filename=package://car_control/meshes/BR_wheel.STL; visual mesh filename=package://car_control/meshes/BR_wheel.STL
- added link dummy_link
- link BL_wheel: geometry collision mesh filename=package://car_control/meshes/BL_wheel.STL; visual mesh filename=package://car_control/meshes/BL_wheel.STL
- link FL_wheel: geometry collision mesh filename=package://car_control/meshes/FL_wheel.STL; visual mesh filename=package://car_control/meshes/FL_wheel.STL
- link FR_wheel: geometry collision mesh filename=package://car_control/meshes/FR_wheel.STL; visual mesh filename=package://car_control/meshes/FR_wheel.STL
- link base_link: geometry collision mesh filename=package://car_control/meshes/base_link.STL; visual mesh filename=package://car_control/meshes/base_link.STL
Joints:
- removed joint BR_coord
- added joint BR_joint: type revolute, parent base_link, child BR_wheel, origin xyz=-0.20624 -0.3302 -0.14111 rpy=0 0 0, axis 0 1 0, limit lower=-1000000 upper=1000000 effort=100 velocity=1000
- added joint dummy_joint: type fixed, parent dummy_link, child base_link
- joint BL_joint: limit effort=1 velocity=1 -> lower=-1000000 upper=1000000 effort=100 velocity=1000; type continuous -> revolute
- joint FL_joint: limit effort=1 velocity=1 -> lower=-1000000 upper=1000000 effort=100 velocity=1000; type continuous -> revolute
- joint FR_joint: limit effort=1 velocity=1 -> lower=-1000000 upper=1000000 effort=100 velocity=1000; type continuous -> revolute

File: urdf/final.urdf (robot description, URDF)
Before this commit: robot , 7 links, 6 joints
Links:
- removed link BR_coord
- added link BR_wheel, mass 2.8186; collision mesh filename=package://car_control/meshes/BR_wheel.STL; visual mesh filename=package://car_control/meshes/BR_wheel.STL
- added link dummy_link
- link BL_wheel: geometry collision mesh filename=package://car_control/meshes/BL_wheel.STL; visual mesh filename=package://car_control/meshes/BL_wheel.STL
- link FL_wheel: geometry collision mesh filename=package://car_control/meshes/FL_wheel.STL; visual mesh filename=package://car_control/meshes/FL_wheel.STL
- link FR_wheel: geometry collision mesh filename=package://car_control/meshes/FR_wheel.STL; visual mesh filename=package://car_control/meshes/FR_wheel.STL
- link base_laser: geometry collision mesh filename=package://car_control/meshes/ydlidar.dae; visual mesh filename=package://car_control/meshes/ydlidar.dae
- link base_link: geometry collision mesh filename=package://car_control/meshes/base_link.STL; visual mesh filename=package://car_control/meshes/base_link.STL
Joints:
- removed joint BR_coord
- removed joint laser_joint_bot
- added joint BR_joint: type revolute, parent base_link, child BR_wheel, origin xyz=-0.20624 -0.3302 -0.14111 rpy=0 0 0, axis 0 1 0, limit lower=-1000000 upper=1000000 effort=10 velocity=100
- added joint dummy_joint: type fixed, parent dummy_link, child base_link
- added joint lidar_joint: type fixed, parent base_link, child base_laser, origin xyz=0 0 0 rpy=0 0 0
- joint BL_joint: limit effort=1 velocity=1 -> lower=-1000000 upper=1000000 effort=10 velocity=100; type continuous -> revolute
- joint FL_joint: limit effort=1 velocity=1 -> lower=-1000000 upper=1000000 effort=10 velocity=100; type continuous -> revolute
- joint FR_joint: limit effort=1 velocity=1 -> lower=-1000000 upper=1000000 effort=10 velocity=100; type continuous -> revolute

File: urdf/my_robot_integration.urdf.xacro (robot description, xacro)
@@ -1,3 +1,12 @@
-<gazebo reference="base_laser">
+<?xml version="1.0"?>
+<!-- Name your robot here -->
+<robot name ="car_control" xmlns:xacro="http://wiki.ros.org/xacro">
+<!-- Include your urdf files here -->
+	<!-- Include Robot's urdf filepath -->
+	<!-- Include Lidar's urdf filepath -->
+	<xacro:include filename="car_control.urdf"/>
+	<xacro:include filename="ydlidar.urdf"/>
+<!-- Add your gazebo sensors here -->
+	<gazebo reference="base_laser">
 		<!-- <gravity>true</gravity> -->
 		<!-- Gazebo has fixed set of Sensors types. Check them out here <> -->
@@ -30,7 +39,28 @@
             <plugin name="gazebo_ros_head_hokuyo_controller" filename="libgazebo_ros_laser.so">
             	<!-- Use topic name as /my_robot/scan -->
-				<topicName></topicName>
+				<topicName>/car_control/scan</topicName>
 				<frameName>laser_frame</frameName>
 			</plugin>
 		</sensor>
 	</gazebo>
+<!--  Gazebo plugin for control here is already added for you -->
+	<gazebo>
+		<plugin name="gazebo_ros_control" filename="libgazebo_ros_control.so">
+			<robotNamespace>/car_control</robotNamespace>
+			<robotSimType>gazebo_ros_control/DefaultRobotHWSim</robotSimType>
+			<legacyModeNS>true</legacyModeNS>
+		</plugin>
+	</gazebo>
+<!-- Create a joint between your robot and sensor -->
+<joint
+    	name="lidar_joint"
+		type="fixed">
+		<origin
+			xyz="0 0 0"
+			rpy="0 0 0"/>
+    	<parent
+     		link="base_link" />
+    	<child
+      		link="base_laser" />
+  	</joint>
+</robot>

File: urdf/ydlidar.urdf (robot description, URDF)
Before this commit: robot ydlidar, 2 links, 1 joints
Links:
- link base_laser: geometry collision mesh filename=package://car_control/meshes/ydlidar.dae; visual mesh filename=package://car_control/meshes/ydlidar.dae
